File: kicad_files/sodiumBMS.kicad_sch (KiCad schematic)
At the start: 23 parts, among them J1 Conn_01x02, J3 USB_C_Receptacle_USB2.0_16P, J4 Conn_02x03_Odd_Even, Q4 AO3400A, SW2 BOOT, SW3 RESET, U1 STM32F446RETx, U4 LM3940, Y1 8MHz or 16 Mhz

Commit message: added some connections for the PD controller
Parts:
- removed R20, R21: 5.1k, Resistor_SMD:R_0805_2012Metric_Pad1.20x1.40mm_HandSolder, symbol Device:R_Small
Connections:
- net CC1: now reaches J3.A5 (CC1)
- net SCL: now reaches U1.61 (PB8)
- net SDA: now reaches U1.62 (PB9)
- net CC2: now reaches J3.B5 (CC2)
- net usb_5v_in renamed VBUS_IN
Other:
- note added: "need to remove this because the LDO will no longer work, probably can get 5 or 3.3V from CYPD"
