File: kicad_files/sodiumBMS.kicad_sch (KiCad schematic)
At the start: 21 parts, among them J1 Conn_01x02, J3 USB_C_Receptacle_USB2.0_16P, J4 Conn_02x03_Odd_Even, Q4 AO3400A, SW2 BOOT, SW3 RESET, U1 STM32F446RETx, U4 LM3940, Y1 8MHz or 16 Mhz

Commit message: fixed some labels and added some passives
Changed lines of the file:
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@@
+	(wire
+		(pts
+			(xy 259.08 40.64) (xy 264.16 40.64)
+		)
+		(stroke
+			(width 0)
+			(type default)
+		)
+	)
 	(wire
 		(pts
@@
 		(pts
 			(xy 191.77 45.72) (xy 191.77 36.83)
+		)
+		(stroke
+			(width 0)
+			(type default)
+		)
+	)
+	(wire
+		(pts
+			(xy 259.08 38.1) (xy 264.16 38.1)
 		)
 		(stroke
@@
 		)
 	)
+	(label "SDA"
+		(at 264.16 38.1 0)
+		(effects
+			(font
+				(size 1.27 1.27)
+			)
+			(justify left bottom)
+		)
+	)
 	(label "CC1"
 		(at 179.07 105.41 180)
@@
 		)
 	)
+	(label "SCL"
+		(at 264.16 40.64 0)
+		(effects
+			(font
+				(size 1.27 1.27)
+			)
+			(justify left bottom)
+		)
+	)

Commit message: Finally finish BQ24172 schematic
Other:
- sheet Charging and Balancing renamed Charging
- sheet Charging ports: added 3V3, status; removed none
Changed lines of the file:
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@@
 			(color 0 0 0 0)
 		)
-		(property "Sheetname" "Charging and Balancing"
+		(property "Sheetname" "Charging"
 			(at 223.52 22.1484 0)
 			(show_name no)
@@
 			(effects
 				(font
+					(size 1.27 1.27)
+				)
+				(justify left)
+			)
+		)
+		(pin "3V3" input
+			(at 223.52 39.37 180)
+			(effects
+				(font
+					(size 1.27 1.27)
+				)
+				(justify left)
+			)
+		)
+		(pin "status" output
+			(at 223.52 43.18 180)
+			(effects
+				(font
